Commit message: Fix xacro file

File: gen2_common/gen2_description/urdf/gen2.xacro (robot description, xacro)
@@ -424,3 +424,22 @@
     </inertial>
   </link>
+<joint name="left_motor_joint" type="fixed">
+    <origin xyz="0.035 0 0.01" rpy="0 0 0" />
+    <parent link="base_link" />
+    <child link="left_motor_link" />
+  </joint>
+<link name="left_motor_link">
+		<inertial>
+			<mass value="1" />
+			<origin xyz=" 0 0 0" />
+			<inertia ixx="1.0" ixy="0.0" ixz="0.0" iyy="1.0" iyz="0.0" izz="1.0" />
+		</inertial>
+		<visual>
+			<origin xyz=" 0 0 0" rpt=" 0 0 0" />
+			<material name="Grey" />
+			<geometry>
+				<cylinder length="0.007" radius="0.2025" />
+			</geometry>
+		</visual>
+	</link>
 </robot>

Commit message: Updated Xacro File

File: gen2_common/gen2_description/urdf/gen2.xacro (robot description, xacro)
@@ -425,5 +425,5 @@
   </link>
 <joint name="left_motor_joint" type="fixed">
-    <origin xyz="0.035 0 0.01" rpy="0 0 0" />
+    <origin xyz="0.0975 0 -0.05" rpy="0 0 0" />
     <parent link="base_link" />
     <child link="left_motor_link" />
@@ -437,7 +437,45 @@
 		<visual>
 			<origin xyz=" 0 0 0" rpt=" 0 0 0" />
-			<material name="Grey" />
-			<geometry>
-				<cylinder length="0.007" radius="0.2025" />
+			<material name="Green" />
+			<geometry>
+				<box size="0.125 0.09 0.10" />
+			</geometry>
+		</visual>
+	</link>
+<joint name="right_motor_joint" type="fixed">
+    <origin xyz="-0.0975 0 -0.045" rpy="0 0 0" />
+    <parent link="base_link" />
+    <child link="right_motor_link" />
+  </joint>
+<link name="right_motor_link">
+		<inertial>
+			<mass value="1" />
+			<origin xyz=" 0 0 0" />
+			<inertia ixx="1.0" ixy="0.0" ixz="0.0" iyy="1.0" iyz="0.0" izz="1.0" />
+		</inertial>
+		<visual>
+			<origin xyz=" 0 0 0" rpt=" 0 0 0" />
+			<material name="Green" />
+			<geometry>
+				<box size="0.125 0.10 0.09" />
+			</geometry>
+		</visual>
+	</link>
+<joint name="left_wheel_joint" type="fixed">
+    <origin xyz="0.0975 0 -0.04" rpy="0 1.6 0" />
+    <parent link="left_motor_link" />
+    <child link="left_wheel_link" />
+  </joint>
+<link name="left_wheel_link">
+		<inertial>
+			<mass value="1" />
+			<origin xyz=" 0 0 0" />
+			<inertia ixx="1.0" ixy="0.0" ixz="0.0" iyy="1.0" iyz="0.0" izz="1.0" />
+		</inertial>
+		<visual>
+			<origin xyz=" 0 0 0" rpt=" 0 0 0" />
+			<material name="Black" />
+			<geometry>
+				 <cylinder length="0.038" radius="0.075" />
 			</geometry>
 		</visual>

Commit message: Working Code Base. PS3 Joystick Working

File: gen2_common/gen2_description/urdf/gen2.xacro (robot description, xacro)
@@ -425,5 +425,5 @@
   </link>
 <joint name="left_motor_joint" type="fixed">
-    <origin xyz="0.0975 0 -0.05" rpy="0 0 0" />
+    <origin xyz=" 0 0.0975 -0.045" rpy="0 0 1.55" />
     <parent link="base_link" />
     <child link="left_motor_link" />
@@ -437,12 +437,12 @@
 		<visual>
 			<origin xyz=" 0 0 0" rpt=" 0 0 0" />
-			<material name="Green" />
-			<geometry>
-				<box size="0.125 0.09 0.10" />
+			<material name="White" />
+			<geometry>
+				<box size="0.125 0.10 0.09" />
 			</geometry>
 		</visual>
 	</link>
 <joint name="right_motor_joint" type="fixed">
-    <origin xyz="-0.0975 0 -0.045" rpy="0 0 0" />
+    <origin xyz="0 -0.0975 -0.045" rpy="0 0 1.575" />
     <parent link="base_link" />
     <child link="right_motor_link" />
@@ -456,5 +456,5 @@
 		<visual>
 			<origin xyz=" 0 0 0" rpt=" 0 0 0" />
-			<material name="Green" />
+			<material name="White" />
 			<geometry>
 				<box size="0.125 0.10 0.09" />
@@ -463,5 +463,5 @@
 	</link>
 <joint name="left_wheel_joint" type="fixed">
-    <origin xyz="0.0975 0 -0.04" rpy="0 1.6 0" />
+    <origin xyz="0.0825 0 -0.035" rpy="0 1.575 0" />
     <parent link="left_motor_link" />
     <child link="left_wheel_link" />
@@ -481,3 +481,98 @@
 		</visual>
 	</link>
+<joint name="right_wheel_joint" type="fixed">
+    <origin xyz="-0.0825 0 -0.035" rpy="0 1.575 0" />
+    <parent link="right_motor_link" />
+    <child link="right_wheel_link" />
+  </joint>
+<link name="right_wheel_link">
+		<inertial>
+			<mass value="1" />
+			<origin xyz=" 0 0 0" />
+			<inertia ixx="1.0" ixy="0.0" ixz="0.0" iyy="1.0" iyz="0.0" izz="1.0" />
+		</inertial>
+		<visual>
+			<origin xyz=" 0 0 0" rpt=" 0 0 0" />
+			<material name="Black" />
+			<geometry>
+				 <cylinder length="0.038" radius="0.075" />
+			</geometry>
+		</visual>
+	</link>
+<joint name="front_castor_base_joint" type="fixed">
+    <origin xyz=" 0.155 0 -0.0325" rpy="0 0 1.55" />
+    <parent link="base_link" />
+    <child link="front_castor_base_link" />
+  </joint>
+<link name="front_castor_base_link">
+		<inertial>
+			<mass value="1" />
+			<origin xyz=" 0 0 0" />
+			<inertia ixx="1.0" ixy="0.0" ixz="0.0" iyy="1.0" iyz="0.0" izz="1.0" />
+		</inertial>
+		<visual>
+			<origin xyz=" 0 0 0" rpt=" 0 0 0" />
+			<material name="White" />
+			<geometry>
+				<box size="0.07 0.05 0.065" />
+			</geometry>
+		</visual>
+	</link>
+<joint name="rear_castor_base_joint" type="fixed">
+    <origin xyz=" -0.155 0 -0.0325" rpy="0 0 1.55" />
+    <parent link="base_link" />
+    <child link="rear_castor_base_link" />
+  </joint>
+<link name="rear_castor_base_link">
+		<inertial>
+			<mass value="1" />
+			<origin xyz=" 0 0 0" />
+			<inertia ixx="1.0" ixy="0.0" ixz="0.0" iyy="1.0" iyz="0.0" izz="1.0" />
+		</inertial>
+		<visual>
+			<origin xyz=" 0 0 0" rpt=" 0 0 0" />
+			<material name="White" />
+			<geometry>
+				<box size="0.07 0.05 0.065" />
+			</geometry>
+		</visual>
+	</link>
+<joint name="front_castor_joint" type="fixed">
+    <origin xyz="0 0 -0.075" rpy="0 1.575 0" />
+    <parent link="front_castor_base_link" />
+    <child link="front_castor_link" />
+  </joint>
+<link name="front_castor_link">
+		<inertial>
+			<mass value="1" />
+			<origin xyz=" 0 0 0" />
+			<inertia ixx="1.0" ixy="0.0" ixz="0.0" iyy="1.0" iyz="0.0" izz="1.0" />
+		</inertial>
+		<visual>
+			<origin xyz=" 0 0 0" rpt=" 0 0 0" />
+			<material name="Black" />
+			<geometry>
+				 <cylinder length="0.02" radius="0.045" />
+			</geometry>
+		</visual>
+	</link>
+<joint name="rear_castor_joint" type="fixed">
+    <origin xyz="0 0 -0.075" rpy="0 1.575 0" />
+    <parent link="rear_castor_base_link" />
+    <child link="rear_castor_link" />
+  </joint>
+<link name="rear_castor_link">
+		<inertial>
+			<mass value="1" />
+			<origin xyz=" 0 0 0" />
+			<inertia ixx="1.0" ixy="0.0" ixz="0.0" iyy="1.0" iyz="0.0" izz="1.0" />
+		</inertial>
+		<visual>
+			<origin xyz=" 0 0 0" rpt=" 0 0 0" />
+			<material name="Black" />
+			<geometry>
+				 <cylinder length="0.02" radius="0.045" />
+			</geometry>
+		</visual>
+	</link>
 </robot>

Commit message: Made change to xacro file to add odom_combined link as a test

File: gen2_common/gen2_description/urdf/gen2.xacro (robot description, xacro)
@@ -87,8 +87,20 @@
 		</visual>
 	</link>
+	<link name="odom_combined">
+		<inertial>
+			<mass value="1" />
+			<origin xyz=" 0 0 0" />
+			<inertia ixx="1.0" ixy="0.0" ixz="0.0" iyy="1.0" iyz="0.0" izz="1.0" />
+		</inertial>
+	</link>
 	<joint name="base_footprint_joint" type="fixed">
 		<origin xyz="0 0 0.15" rpy="0 0 0" />
 		<parent link="base_footprint" />
 		<child link="base_link" />
+	</joint>
+	<joint name="odom_combined_joint" type="fixed">
+		<origin xyz="0 0 0.15" rpy="0 0 0" />
+		<parent link="base_footprint" />
+		<child link="odom_combined" />
 	</joint>
 	<joint name="base_middle_joint" type="fixed">

Commit message: Removed odom_combined from xacro file

File: gen2_common/gen2_description/urdf/gen2.xacro (robot description, xacro)
@@ -87,20 +87,8 @@
 		</visual>
 	</link>
-	<link name="odom_combined">
-		<inertial>
-			<mass value="1" />
-			<origin xyz=" 0 0 0" />
-			<inertia ixx="1.0" ixy="0.0" ixz="0.0" iyy="1.0" iyz="0.0" izz="1.0" />
-		</inertial>
-	</link>
 	<joint name="base_footprint_joint" type="fixed">
 		<origin xyz="0 0 0.15" rpy="0 0 0" />
 		<parent link="base_footprint" />
 		<child link="base_link" />
-	</joint>
-	<joint name="odom_combined_joint" type="fixed">
-		<origin xyz="0 0 0.15" rpy="0 0 0" />
-		<parent link="base_footprint" />
-		<child link="odom_combined" />
 	</joint>
 	<joint name="base_middle_joint" type="fixed">

Commit message: Made changes to USRF in order to fix loop in tree.

File: gen2_common/gen2_description/urdf/gen2.xacro (robot description, xacro)
@@ -7,4 +7,5 @@
   <property name="base_x" value="0.33" />
   <property name="base_y" value="0.33" />
+<!-- Material colors for reference -->
 	<material name="Green">
 		<color rgba="0.0 0.8 0.0 1.0"/>
@@ -25,4 +26,5 @@
 		<color rgba="0.25 0.25 0.25 1.0"/>
 	</material>
+<!-- base plate links and joints -->
 	<link name="base_footprint">
 	    <inertial>
@@ -102,30 +104,350 @@
 		<child link="base_top_link" />
 	</joint>
+<!-- front left bar link and joints -->
+  <link name="middle_fl_link">
+    <visual>
+      <geometry>
+        <cylinder length="0.25" radius="0.01" />
+      </geometry>
+      <material name="White" />
+    </visual>
+    <inertial>
+      <mass value="0.000001" />
+      <origin xyz="0 0 0" />
+      <inertia ixx="0.0001" ixy="0.0" ixz="0.0"
+        iyy="0.0001" iyz="0.0"
+        izz="0.0001" />
+    </inertial>
+  </link>
+  <link name="top_fl_link">
+    <visual>
+      <geometry>
+        <cylinder length="0.125" radius="0.01" />
+      </geometry>
+      <material name="White" />
+    </visual>
+    <inertial>
+      <mass value="0.000001" />
+      <origin xyz="0 0 0" />
+      <inertia ixx="0.0001" ixy="0.0" ixz="0.0"
+        iyy="0.0001" iyz="0.0"
+        izz="0.0001" />
+    </inertial>
+  </link>
+<joint name="middle_fl_joint" type="fixed">
+    <origin xyz="0.14 0.13 0.125" rpy="0 0 0" />
+    <parent link="base_link" />
+    <child link="middle_fl_link" />
+  </joint>
+<joint name="top_fl_joint" type="fixed">
+    <origin xyz="0.14 0.13 0.0625" rpy="0 0 0" />
+    <parent link="middle_fl_link" />
+    <child link="top_fl_link" />
+  </joint>
+<!-- front right link and joints -->
+  <link name="middle_fr_link">
+    <visual>
+      <geometry>
+        <cylinder length="0.25" radius="0.01" />
+      </geometry>
+      <material name="White" />
+    </visual>
+    <inertial>
+      <mass value="0.000001" />
+      <origin xyz="0 0 0" />
+      <inertia ixx="0.0001" ixy="0.0" ixz="0.0"
+        iyy="0.0001" iyz="0.0"
+        izz="0.0001" />
+    </inertial>
+  </link>
+  <link name="top_fr_link">
+    <visual>
+      <geometry>
+        <cylinder length="0.125" radius="0.01" />
+      </geometry>
+      <material name="White" />
+    </visual>
+    <inertial>
+      <mass value="0.000001" />
+      <origin xyz="0 0 0" />
+      <inertia ixx="0.0001" ixy="0.0" ixz="0.0"
+        iyy="0.0001" iyz="0.0"
+        izz="0.0001" />
+    </inertial>
+  </link>
+<joint name="middle_fr_joint" type="fixed">
+    <origin xyz="0.14 -0.13 0.125" rpy="0 0 0" />
+    <parent link="base_link" />
+    <child link="middle_fr_link" />
+  </joint>
+<joint name="top_fr_joint" type="fixed">
+    <origin xyz="0.14 -0.13 0.0625" rpy="0 0 0" />
+    <parent link="middle_fr_link" />
+    <child link="top_fr_link" />
+  </joint>
+<!-- rear left bar links and joints -->
+  <link name="middle_rl_link">
+    <visual>
+      <geometry>
+        <cylinder length="0.25" radius="0.01" />
+      </geometry>
+      <material name="White" />
+    </visual>
+    <inertial>
+      <mass value="0.000001" />
+      <origin xyz="0 0 0" />
+      <inertia ixx="0.0001" ixy="0.0" ixz="0.0"
+        iyy="0.0001" iyz="0.0"
+        izz="0.0001" />
+    </inertial>
+  </link>
+  <link name="top_rl_link">
+    <visual>
+      <geometry>
+        <cylinder length="0.125" radius="0.01" />
+      </geometry>
+      <material name="White" />
+    </visual>
+    <inertial>
+      <mass value="0.000001" />
+      <origin xyz="0 0 0" />
+      <inertia ixx="0.0001" ixy="0.0" ixz="0.0"
+        iyy="0.0001" iyz="0.0"
+        izz="0.0001" />
+    </inertial>
+  </link>
+<joint name="middle_rl_joint" type="fixed">
+    <origin xyz="-0.14 0.13 0.125" rpy="0 0 0" />
+    <parent link="base_link" />
+    <child link="middle_rl_link" />
+  </joint>
+<joint name="top_rl_joint" type="fixed">
+    <origin xyz="-0.14 0.13 0.0625" rpy="0 0 0" />
+    <parent link="middle_rl_link" />
+    <child link="top_rl_link" />
+  </joint>
+<!-- rear right bar links and joints -->
+  <link name="middle_rr_link">
+    <visual>
+      <geometry>
+        <cylinder length="0.25" radius="0.01" />
+      </geometry>
+      <material name="White" />
+    </visual>
+    <inertial>
+      <mass value="0.000001" />
+      <origin xyz="0 0 0" />
+      <inertia ixx="0.0001" ixy="0.0" ixz="0.0"
+        iyy="0.0001" iyz="0.0"
+        izz="0.0001" />
+    </inertial>
+  </link>
+  <link name="top_rr_link">
+    <visual>
+      <geometry>
+        <cylinder length="0.125" radius="0.01" />
+      </geometry>
+      <material name="White" />
+    </visual>
+    <inertial>
+      <mass value="0.000001" />
+      <origin xyz="0 0 0" />
+      <inertia ixx="0.0001" ixy="0.0" ixz="0.0"
+        iyy="0.0001" iyz="0.0"
+        izz="0.0001" />
+    </inertial>
+  </link>
+<joint name="middle_rr_joint" type="fixed">
+    <origin xyz="-0.14 -0.13 0.125" rpy="0 0 0" />
+    <parent link="base_link" />
+    <child link="middle_rr_link" />
+  </joint>
+<joint name="top_rr_joint" type="fixed">
+    <origin xyz="-0.14 -0.13 0.0625" rpy="0 0 0" />
+    <parent link="middle_rr_link" />
+    <child link="top_rr_link" />
+  </joint>
+<!-- motor links and joints -->
+<link name="left_motor_link">
+		<inertial>
+			<mass value="1" />
+			<origin xyz=" 0 0 0" />
+			<inertia ixx="1.0" ixy="0.0" ixz="0.0" iyy="1.0" iyz="0.0" izz="1.0" />
+		</inertial>
+		<visual>
+			<origin xyz=" 0 0 0" rpt=" 0 0 0" />
+			<material name="White" />
+			<geometry>
+				<box size="0.125 0.10 0.09" />
+			</geometry>
+		</visual>
+	</link>
+<joint name="left_motor_joint" type="fixed">
+    <origin xyz=" 0 0.0975 -0.045" rpy="0 0 1.55" />
+    <parent link="base_link" />
+    <child link="left_motor_link" />
+  </joint>
+<link name="right_motor_link">
+		<inertial>
+			<mass value="1" />
+			<origin xyz=" 0 0 0" />
+			<inertia ixx="1.0" ixy="0.0" ixz="0.0" iyy="1.0" iyz="0.0" izz="1.0" />
+		</inertial>
+		<visual>
+			<origin xyz=" 0 0 0" rpt=" 0 0 0" />
+			<material name="White" />
+			<geometry>
+				<box size="0.125 0.10 0.09" />
+			</geometry>
+		</visual>
+	</link>
+<joint name="right_motor_joint" type="fixed">
+    <origin xyz="0 -0.0975 -0.045" rpy="0 0 1.575" />
+    <parent link="base_link" />
+    <child link="right_motor_link" />
+  </joint>
+<!-- wheel links and joints -->
+<link name="left_wheel_link">
+		<inertial>
+			<mass value="1" />
+			<origin xyz=" 0 0 0" />
+			<inertia ixx="1.0" ixy="0.0" ixz="0.0" iyy="1.0" iyz="0.0" izz="1.0" />
+		</inertial>
+		<visual>
+			<origin xyz=" 0 0 0" rpt=" 0 0 0" />
+			<material name="Black" />
+			<geometry>
+				 <cylinder length="0.038" radius="0.075" />
+			</geometry>
+		</visual>
+	</link>
+<joint name="left_wheel_joint" type="fixed">
+    <origin xyz="0.0825 0 -0.035" rpy="0 1.575 0" />
+    <parent link="left_motor_link" />
+    <child link="left_wheel_link" />
+  </joint>
+<link name="right_wheel_link">
+		<inertial>
+			<mass value="1" />
+			<origin xyz=" 0 0 0" />
+			<inertia ixx="1.0" ixy="0.0" ixz="0.0" iyy="1.0" iyz="0.0" izz="1.0" />
+		</inertial>
+		<visual>
+			<origin xyz=" 0 0 0" rpt=" 0 0 0" />
+			<material name="Black" />
+			<geometry>
+				 <cylinder length="0.038" radius="0.075" />
+			</geometry>
+		</visual>
+	</link>
+<joint name="right_wheel_joint" type="fixed">
+    <origin xyz="-0.0825 0 -0.035" rpy="0 1.575 0" />
+    <parent link="right_motor_link" />
+    <child link="right_wheel_link" />
+  </joint>
+<!-- castor links and joints -->
+<joint name="front_castor_base_joint" type="fixed">
+    <origin xyz=" 0.155 0 -0.0325" rpy="0 0 1.55" />
+    <parent link="base_link" />
+    <child link="front_castor_base_link" />
+  </joint>
+<link name="front_castor_base_link">
+		<inertial>
+			<mass value="1" />
+			<origin xyz=" 0 0 0" />
+			<inertia ixx="1.0" ixy="0.0" ixz="0.0" iyy="1.0" iyz="0.0" izz="1.0" />
+		</inertial>
+		<visual>
+			<origin xyz=" 0 0 0" rpt=" 0 0 0" />
+			<material name="White" />
+			<geometry>
+				<box size="0.07 0.05 0.065" />
+			</geometry>
+		</visual>
+	</link>
+<joint name="rear_castor_base_joint" type="fixed">
+    <origin xyz=" -0.155 0 -0.0325" rpy="0 0 1.55" />
+    <parent link="base_link" />
+    <child link="rear_castor_base_link" />
+  </joint>
+<link name="rear_castor_base_link">
+		<inertial>
+			<mass value="1" />
+			<origin xyz=" 0 0 0" />
+			<inertia ixx="1.0" ixy="0.0" ixz="0.0" iyy="1.0" iyz="0.0" izz="1.0" />
+		</inertial>
+		<visual>
+			<origin xyz=" 0 0 0" rpt=" 0 0 0" />
+			<material name="White" />
+			<geometry>
+				<box size="0.07 0.05 0.065" />
+			</geometry>
+		</visual>
+	</link>
+<joint name="front_castor_joint" type="fixed">
+    <origin xyz="0 0 -0.075" rpy="0 1.575 0" />
+    <parent link="front_castor_base_link" />
+    <child link="front_castor_link" />
+  </joint>
+<link name="front_castor_link">
+		<inertial>
+			<mass value="1" />
+			<origin xyz=" 0 0 0" />
+			<inertia ixx="1.0" ixy="0.0" ixz="0.0" iyy="1.0" iyz="0.0" izz="1.0" />
+		</inertial>
+		<visual>
+			<origin xyz=" 0 0 0" rpt=" 0 0 0" />
+			<material name="Black" />
+			<geometry>
+				 <cylinder length="0.02" radius="0.045" />
+			</geometry>
+		</visual>
+	</link>
+<joint name="rear_castor_joint" type="fixed">
+    <origin xyz="0 0 -0.075" rpy="0 1.575 0" />
+    <parent link="rear_castor_base_link" />
+    <child link="rear_castor_link" />
+  </joint>
+<link name="rear_castor_link">
+		<inertial>
+			<mass value="1" />
+			<origin xyz=" 0 0 0" />
+			<inertia ixx="1.0" ixy="0.0" ixz="0.0" iyy="1.0" iyz="0.0" izz="1.0" />
+		</inertial>
+		<visual>
+			<origin xyz=" 0 0 0" rpt=" 0 0 0" />
+			<material name="Black" />
+			<geometry>
+				 <cylinder length="0.02" radius="0.045" />
+			</geometry>
+		</visual>
+	</link>
+<!-- kinnect links and joints -->
 	<joint name="base_kinect_joint" type="fixed">
-    <origin xyz="0.14 0 0.055" rpy="0 0 0" />
-    <parent link="base_middle_link" />
-    <child link="kinect_link" />
-  </joint>
-  <link name="kinect_link">
-    <inertial>
-      <mass value="0.00001" />
-      <origin xyz="0 0 0" />
-      <inertia ixx="1.0" ixy="0.0" ixz="0.0"
-        iyy="1.0" iyz="0.0"
-        izz="1.0" />
-    </inertial>
-    <visual>
-      <origin xyz=" 0 0 0 " rpy="0 0 0" />
-      <geometry>
-        <mesh filename="package://gen2_description/meshes/kinect.dae"/>
-      </geometry>
-    </visual>
-    <collision>
-      <origin xyz="0.0 0.0 0.0" rpy="0 0 0" />
-      <geometry>
-        <box size="0.0730 .2760 0.0720"/>
-      </geometry>
-    </collision>
-  </link>
+  	        <origin xyz="0.14 0 0.055" rpy="0 0 0" />
+ 	        <parent link="base_middle_link" />
+                <child link="kinect_link" />
+       </joint>
+       <link name="kinect_link">
+         <inertial>
+          <mass value="0.00001" />
+          <origin xyz="0 0 0" />
+         <inertia ixx="1.0" ixy="0.0" ixz="0.0"
+                            iyy="1.0" iyz="0.0"
+                            izz="1.0" />
+         </inertial>
+        <visual>
+         <origin xyz=" 0 0 0 " rpy="0 0 0" />
+          <geometry>
+          <mesh filename="package://gen2_description/meshes/kinect.dae"/>
+          </geometry>
+        </visual>
+        <collision>
+         <origin xyz="0.0 0.0 0.0" rpy="0 0 0" />
+         <geometry>
+          <box size="0.0730 .2760 0.0720"/>
+         </geometry>
+        </collision>
+         </link>
   <joint name="kinect_depth_joint" type="fixed">
     <origin xyz="0 0.018 0" rpy="0 0 0" />
@@ -184,4 +506,5 @@
     </inertial>
   </link>
+<!-- Gyro link and joint -->
 <joint name="gyro_joint" type="fixed">
     <origin xyz="0 0.03 0.01" rpy="0 0 0" />
@@ -204,4 +527,5 @@
     </inertial>
   </link>
+<!--laser link and joint -->
  <joint name="laser_joint" type="fixed">
     <origin xyz="-0.065 0 0.075" rpy="0 0 0" />
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
Commit message: Fixed error in urdf

File: gen2_common/gen2_description/urdf/gen2.xacro (robot description, xacro)
@@ -141,5 +141,5 @@
   </joint>
 <joint name="top_fl_joint" type="fixed">
-    <origin xyz="0.14 0.13 0.0625" rpy="0 0 0" />
+    <origin xyz="0 0 0.0625" rpy="0 0 0" />
     <parent link="middle_fl_link" />
     <child link="top_fl_link" />
@@ -182,5 +182,5 @@
   </joint>
 <joint name="top_fr_joint" type="fixed">
-    <origin xyz="0.14 -0.13 0.0625" rpy="0 0 0" />
+    <origin xyz="0 0 0.0625" rpy="0 0 0" />
     <parent link="middle_fr_link" />
     <child link="top_fr_link" />
@@ -223,5 +223,5 @@
   </joint>
 <joint name="top_rl_joint" type="fixed">
-    <origin xyz="-0.14 0.13 0.0625" rpy="0 0 0" />
+    <origin xyz="0 0 0.0625" rpy="0 0 0" />
     <parent link="middle_rl_link" />
     <child link="top_rl_link" />
@@ -264,5 +264,5 @@
   </joint>
 <joint name="top_rr_joint" type="fixed">
-    <origin xyz="-0.14 -0.13 0.0625" rpy="0 0 0" />
+    <origin xyz="0 0 0.0625" rpy="0 0 0" />
     <parent link="middle_rr_link" />
     <child link="top_rr_link" />

Commit message: Fixed error in urdf

File: gen2_common/gen2_description/urdf/gen2.xacro (robot description, xacro)
@@ -141,5 +141,5 @@
   </joint>
 <joint name="top_fl_joint" type="fixed">
-    <origin xyz="0 0 0.0625" rpy="0 0 0" />
+    <origin xyz="0 0 0.1875" rpy="0 0 0" />
     <parent link="middle_fl_link" />
     <child link="top_fl_link" />
@@ -182,5 +182,5 @@
   </joint>
 <joint name="top_fr_joint" type="fixed">
-    <origin xyz="0 0 0.0625" rpy="0 0 0" />
+    <origin xyz="0 0 0.1875" rpy="0 0 0" />
     <parent link="middle_fr_link" />
     <child link="top_fr_link" />
@@ -223,5 +223,5 @@
   </joint>
 <joint name="top_rl_joint" type="fixed">
-    <origin xyz="0 0 0.0625" rpy="0 0 0" />
+    <origin xyz="0 0 0.1875" rpy="0 0 0" />
     <parent link="middle_rl_link" />
     <child link="top_rl_link" />
@@ -264,5 +264,5 @@
   </joint>
 <joint name="top_rr_joint" type="fixed">
-    <origin xyz="0 0 0.0625" rpy="0 0 0" />
+    <origin xyz="0 0 0.1875" rpy="0 0 0" />
     <parent link="middle_rr_link" />
     <child link="top_rr_link" />
